File: schematic/rpi_cpld.kicad_pcb (KiCad board)
At the start: 2 copper layers, 65 x 56.5 mm, 87 parts, among them J1 CONN_02, J2 RPi_Hat-rescue_RPi_GPIO, J3 , J4 Conn_01x10, J5 UART, J6 , J7 I2C, J8 Conn_01x10, J9 , Q1 BC817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

Commit message: new
Parts:
- removed TP1: CLK ext, TestPoint:TestPoint_Loop_D1.80mm_Drill1.0mm_Beaded
Connections:
- J2 pad 1: (no net) -> Net-(J2-Pad1)
- J2 pad 11: (no net) -> Net-(J2-Pad11)
- J2 pad 12: (no net) -> Net-(J2-Pad12)
- J2 pad 17: (no net) -> Net-(J2-Pad17)
- J2 pad 24: (no net) -> Net-(J2-Pad24)
- J2 pad 29: (no net) -> Net-(J2-Pad29)
- J2 pad 37: (no net) -> Net-(J2-Pad37)
- U2 pad 12: (no net) -> Net-(U2-Pad12)
- U2 pad 14: (no net) -> Net-(U2-Pad14)
- U2 pad 15: (no net) -> Net-(U2-Pad15)
- U2 pad 16: (no net) -> Net-(U2-Pad16)
- U2 pad 17: (no net) -> Net-(U2-Pad17)
- U2 pad 18: (no net) -> Net-(U2-Pad18)
- U2 pad 19: (no net) -> Net-(U2-Pad19)
- U2 pad 20: (no net) -> Net-(U2-Pad20)
- U2 pad 21: (no net) -> Net-(U2-Pad21)
- U2 pad 35: (no net) -> Net-(U2-Pad35)
- U2 pad 36: (no net) -> Net-(U2-Pad36)
- U2 pad 38: (no net) -> Net-(U2-Pad38)
- U2 pad 44: (no net) -> Net-(U2-Pad44)
- U2 pad 66: (no net) -> Net-(U2-Pad66)
- U2 pad 67: (no net) -> Net-(U2-Pad67)
- U2 pad 68: (no net) -> Net-(U2-Pad68)
- U2 pad 69: (no net) -> Net-(U2-Pad69)
- U2 pad 70: (no net) -> Net-(U2-Pad70)
- U2 pad 71: (no net) -> Net-(U2-Pad71)
- U2 pad 8: (no net) -> Net-(U2-Pad8)
- U2 pad 81: (no net) -> Net-(U2-Pad81)
- U2 pad 82: (no net) -> Net-(U2-Pad82)
- U2 pad 83: (no net) -> Net-(U2-Pad83)
- U2 pad 84: (no net) -> Net-(U2-Pad84)
- U2 pad 85: (no net) -> Net-(U2-Pad85)
- U2 pad 86: (no net) -> Net-(U2-Pad86)
- U2 pad 87: (no net) -> Net-(U2-Pad87)
- U2 pad 89: (no net) -> Net-(U2-Pad89)
- Y1 pad 1: (no net) -> Net-(Y1-Pad1)
Routing:
- net Net-(U2-Pad62): track 4.52 -> 0.00 mm

Commit message: add
Parts:
- added R38: 1k, Capacitors_SMD:C_0603_HandSoldering, F.Cu at (130.5, 87.7)
- added R39: 1k, Capacitors_SMD:C_0603_HandSoldering, F.Cu at (130.5, 91.2)
- added R40: 1k, Capacitors_SMD:C_0603_HandSoldering, F.Cu at (130.5, 94.7)
- added R41: 1k, Capacitors_SMD:C_0603_HandSoldering, F.Cu at (130.6, 98.3)
- added R42: 1k, Capacitors_SMD:C_0603_HandSoldering, F.Cu at (130.6, 101.8)
- added R43: 1k, Capacitors_SMD:C_0603_HandSoldering, F.Cu at (130.6, 105.3)

Commit message: update
Parts:
- removed the G*** at (100.8, 83.3)
- removed the G*** at (101.2, 72.4)
- added G***: LOGO, schematic:logo_emc2, F.Cu at (101.1, 73.0)
- added G***: LOGO, schematic:logo_rpi, F.Cu at (101.2, 83.2)
- added R44: 0, Capacitors_SMD:C_0603_HandSoldering, B.Cu at (126.6, 105.3)
- renumbered REF** to REF00, REF** to REF01, REF** to REF02
Connections:
- J2 pad 1: Net-(J2-Pad1) -> (no net)
- J2 pad 11: Net-(J2-Pad11) -> (no net)
- J2 pad 12: Net-(J2-Pad12) -> (no net)
- J2 pad 17: Net-(J2-Pad17) -> (no net)
- J2 pad 24: Net-(J2-Pad24) -> (no net)
- J2 pad 29: Net-(J2-Pad29) -> (no net)
- J2 pad 37: Net-(J2-Pad37) -> (no net)
- R38 pad 2: +5V -> Net-(R38-Pad2)
- R39 pad 2: +5V -> Net-(R38-Pad2)
- R40 pad 2: +5V -> Net-(R38-Pad2)
- R41 pad 2: +5V -> Net-(R38-Pad2)
- R42 pad 2: +5V -> Net-(R38-Pad2)
- R43 pad 2: +5V -> Net-(R38-Pad2)
- U2 pad 12: Net-(U2-Pad12) -> (no net)
- U2 pad 14: Net-(U2-Pad14) -> (no net)
- U2 pad 15: Net-(U2-Pad15) -> (no net)
- U2 pad 16: Net-(U2-Pad16) -> (no net)
- U2 pad 17: Net-(U2-Pad17) -> (no net)
- U2 pad 18: Net-(U2-Pad18) -> (no net)
- U2 pad 19: Net-(U2-Pad19) -> (no net)
- U2 pad 20: Net-(U2-Pad20) -> (no net)
- U2 pad 21: Net-(U2-Pad21) -> (no net)
- U2 pad 35: Net-(U2-Pad35) -> (no net)
- U2 pad 36: Net-(U2-Pad36) -> (no net)
- U2 pad 38: Net-(U2-Pad38) -> (no net)
- U2 pad 44: Net-(U2-Pad44) -> (no net)
- U2 pad 62: Net-(U2-Pad62) -> (no net)
- U2 pad 66: Net-(U2-Pad66) -> (no net)
- U2 pad 67: Net-(U2-Pad67) -> (no net)
- U2 pad 68: Net-(U2-Pad68) -> (no net)
- U2 pad 69: Net-(U2-Pad69) -> (no net)
- U2 pad 70: Net-(U2-Pad70) -> (no net)
- U2 pad 71: Net-(U2-Pad71) -> (no net)
- U2 pad 8: Net-(U2-Pad8) -> (no net)
- U2 pad 81: Net-(U2-Pad81) -> (no net)
- U2 pad 82: Net-(U2-Pad82) -> (no net)
- U2 pad 83: Net-(U2-Pad83) -> (no net)
- U2 pad 84: Net-(U2-Pad84) -> (no net)
- U2 pad 85: Net-(U2-Pad85) -> (no net)
- U2 pad 86: Net-(U2-Pad86) -> (no net)
- U2 pad 87: Net-(U2-Pad87) -> (no net)
- U2 pad 89: Net-(U2-Pad89) -> (no net)
- Y1 pad 1: Net-(Y1-Pad1) -> (no net)
Routing:
- net Net-(R38-Pad2): track 0.00 -> 28.9 mm, vias 0 -> 1
- net Net-(J4-Pad7): track 3.88 -> 6.61 mm, vias 0 -> 1
- net Net-(J4-Pad6): track 3.39 -> 5.89 mm, vias 0 -> 1
- net Net-(J4-Pad5): track 3.24 -> 4.57 mm, vias 0 -> 1
- net +5V: track 129.9 -> 131.0 mm
- net Net-(J4-Pad2): track 5.37 -> 6.24 mm, vias 0 -> 1
- net Net-(J4-Pad3): track 3.95 -> 4.73 mm, vias 0 -> 1
- net Net-(J4-Pad4): track 3.71 -> 4.47 mm, vias 0 -> 1
Other:
- board text added: "Pi HAT CNC v2"
- board text removed: "Pi HAT CNC"
