File: schematic/rpi_cpld.sch (KiCad schematic (older format))
At the start: 82 parts, among them J1 CONN_02, J2 RPi_Hat-rescue_RPi_GPIO, J3 , J4 Conn_01x10, J5 UART, J6 , J7 I2C, J8 Conn_01x10, J9 , Q1 BC817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

Commit message: new
Parts:
- removed TP1: CLK ext, TestPoint:TestPoint_Loop_D1.80mm_Drill1.0mm_Beaded, symbol TEST
Changed lines of the file:
@@
-$EndComp
-$Comp
-L TEST TP1
-U 1 1 5C194D56
-P 8630 2520
-F 0 "TP1" V 8630 2820 50  0000 C BNN
-F 1 "CLK ext" V 8605 3075 50  0000 C CNN
-F 2 "TestPoint:TestPoint_Loop_D1.80mm_Drill1.0mm_Beaded" H 8630 2520 50  0001 C CNN
-F 3 "" H 8630 2520 50  0001 C CNN
-	1    8630 2520
-	0    1    1    0
 $EndComp
 $Comp
@@
 U 1 1 5C1AFE11
 P 12135 8035
-F 0 "R32" H 12245 7975 45  0000 L BNN
-F 1 "0" H 11935 7975 45  0000 L BNN
+F 0 "R32" H 12190 8190 45  0000 L BNN
+F 1 "0" H 12075 8190 45  0000 L BNN
 F 2 "Capacitors_SMD:C_0603_HandSoldering" H 12135 8185 20  0001 C CNN
 F 3 "" H 12135 8035 60  0001 C CNN
@@
 $EndComp
 NoConn ~ 6430 2220
-NoConn ~ 11170 3495
 $Comp
 L RESISTOR0805 R33
@@
 $EndComp
 Wire Wire Line
-	2350 1200 2725 1200
-Wire Wire Line
-	2725 1200 3095 1200
-Wire Wire Line
-	3095 1200 3490 1200
+	2350 1200 3490 1200
 Connection ~ 2725 1200
 Wire Wire Line
@@
 Connection ~ 3095 1200
 Wire Wire Line
-	3490 1205 3825 1205
-Wire Wire Line
-	3825 1205 3905 1205
+	3490 1205 3905 1205
 Wire Wire Line
 	3825 1205 3825 1200
 Wire Wire Line
-	3395 900  3490 900
-Wire Wire Line
-	3490 900  3825 900
-Wire Wire Line
-	3825 900  3920 900
-Wire Wire Line
-	2350 900  2725 900
-Wire Wire Line
-	2725 900  2795 900
+	3395 900  3920 900
+Wire Wire Line
+	2350 900  2795 900
 Connection ~ 2725 900
 Connection ~ 3490 900
@@
 	4270 3985 4135 3985
 Wire Wire Line
-	4270 2585 4270 3285
-Wire Wire Line
-	4270 3285 4270 3785
-Wire Wire Line
-	4270 3785 4270 3985
-Wire Wire Line
-	4270 3985 4270 4440
+	4270 4440 4270 2585
 Wire Wire Line
 	4270 3285 4135 3285
@@
 Connection ~ 2145 3585
 Wire Wire Line
-	2145 2785 2145 3585
-Wire Wire Line
-	2145 3585 2145 4285
-Wire Wire Line
-	2145 4285 2145 4440
-Wire Wire Line
-	2145 4440 3050 4440
-Wire Wire Line
-	3050 4440 4270 4440
+	2145 2785 2145 4440
+Wire Wire Line
+	2145 4440 4270 4440
 Connection ~ 2145 4285
 Connection ~ 4270 3985
@@
 Connection ~ 3490 1200
 Wire Wire Line
-	5670 775  5910 775
-Wire Wire Line
-	5910 775  6180 775
-Wire Wire Line
-	6180 775  6430 775
-Wire Wire Line
-	6430 775  6680 775
-Wire Wire Line
-	6680 775  6925 775
+	5670 775  6925 775
 Connection ~ 6180 775
 Connection ~ 6430 775
 Wire Wire Line
-	5670 1075 5910 1075
-Wire Wire Line
-	5910 1075 6180 1075
-Wire Wire Line
-	6180 1075 6305 1075
-Wire Wire Line
-	6305 1075 6430 1075
-Wire Wire Line
-	6430 1075 6680 1075
-Wire Wire Line
-	6680 1075 6925 1075
+	5670 1075 6925 1075
 Connection ~ 6180 1075
 Connection ~ 6430 1075
@@
 	5930 5520 6430 5520
 Wire Wire Line
-	5435 5970 5585 5970
-Wire Wire Line
-	5585 5970 5685 5970
-Wire Wire Line
-	5685 5970 5930 5970
+	5435 5970 5930 5970
 Connection ~ 5685 5970
 Connection ~ 5585 5970
 Wire Wire Line
-	7030 5920 7130 5920
-Wire Wire Line
-	7130 5920 7230 5920
-Wire Wire Line
-	7230 5920 7330 5920
-Wire Wire Line
-	7375 5920 7430 5920
-Wire Wire Line
-	7430 5920 7530 5920
-Wire Wire Line
-	7530 5920 7630 5920
-Wire Wire Line
-	7630 5920 7730 5920
-Wire Wire Line
-	7730 5920 7830 5920
-Wire Wire Line
-	7830 5920 7930 5920
+	7030 5920 7930 5920
 Connection ~ 7130 5920
 Connection ~ 7230 5920
@@
 	2680 7310 2680 6965
 Wire Wire Line
-	2680 6965 3115 6965
-Wire Wire Line
-	3115 6965 3890 6965
+	2680 6965 3890 6965
 Wire Wire Line
 	2680 7410 2830 7410
@@
 	3030 8205 3880 8205
 Wire Wire Line
-	3120 6965 3120 7375
-Wire Wire Line
-	3120 7375 3120 7795
+	3120 6965 3120 7795
 Wire Wire Line
 	3120 6965 3115 6965
@@
 	4490 7165 4705 7165
 Wire Wire Line
-	4705 7165 4705 7575
-Wire Wire Line
-	4705 7575 4705 7995
-Wire Wire Line
-	4705 7995 4705 8405
-Wire Wire Line
-	4705 8405 4705 8830
+	4705 7165 4705 8830
 Wire Wire Line
 	4705 8405 4480 8405
@@
 	9935 7935 9935 8300
 Wire Wire Line
-	9935 8300 10335 8300
-Wire Wire Line
-	10335 8300 10735 8300
-Wire Wire Line
-	10735 8300 10945 8300
-Wire Wire Line
-	10945 8300 11135 8300
-Wire Wire Line
-	11135 8300 11535 8300
-Wire Wire Line
-	11535 8300 11935 8300
-Wire Wire Line
-	11935 8300 11935 8040
-Wire Wire Line
-	11935 8040 11935 7435
+	11935 8300 9935 8300
+Wire Wire Line
+	11935 7435 11935 8300
 Wire Wire Line
 	10335 7835 10335 8300
@@
 Connection ~ 3825 1205
 Wire Wire Line
-	6175 5975 6680 5975
-Wire Wire Line
-	6680 5975 7030 5975
+	6175 5975 7030 5975
 Wire Wire Line
 	7030 5975 7030 5920
@@
 	4305 1205 4305 1260
 Wire Wire Line
-	4305 1260 4665 1260
-Wire Wire Line
-	4665 1260 5120 1260
+	4305 1260 5120 1260
 Wire Wire Line
 	5120 1260 5120 1100
@@
 	5930 5570 5930 5520
 Wire Wire Line
-	7030 1275 7130 1275
-Wire Wire Line
-	7130 1275 7230 1275
-Wire Wire Line
-	7230 1275 7330 1275
-Wire Wire Line
-	7330 1275 7430 1275
-Wire Wire Line
-	7430 1275 7530 1275
-Wire Wire Line
-	7530 1275 7630 1275
-Wire Wire Line
-	7630 1275 7730 1275
-Wire Wire Line
-	7730 1275 7830 1275
-Wire Wire Line
-	7830 1275 7930 1275
+	7030 1275 7930 1275
 Wire Wire Line
 	7930 1275 7930 1320
@@
 	4270 2485 4135 2485
 Wire Wire Line
-	4270 2355 4270 2385
-Wire Wire Line
-	4270 2385 4270 2485
+	4270 2355 4270 2485
 Wire Wire Line
 	4135 2385 4270 2385
@@
 	6345 7940 6345 8305
 Wire Wire Line
-	6345 8305 6745 8305
-Wire Wire Line
-	6745 8305 7145 8305
-Wire Wire Line
-	7145 8305 7355 8305
-Wire Wire Line
-	7355 8305 7545 8305
-Wire Wire Line
-	7545 8305 7945 8305
+	6345 8305 7945 8305
 Wire Wire Line
 	6745 7840 6745 8305
@@
 	5255 6965 5290 6965
 Wire Wire Line
-	5290 6940 5290 6965
-Wire Wire Line
-	5290 6965 5290 7375
-Wire Wire Line
-	5290 7375 5290 7795
-Wire Wire Line
-	5290 7795 5290 8205
-Wire Wire Line
-	5290 8205 5290 8630
+	5290 6940 5290 8630
 Wire Wire Line
 	5290 8630 5255 8630
@@
 	-1   0    0    -1
 $EndComp
-Wire Wire Line
-	7330 5920 7375 5920
+NoConn ~ 8630 2520
 $EndSCHEMATC

Commit message: add
Parts:
- added R38, R39, R40, R41, R42, R43: 1k, Capacitors_SMD:C_0603_HandSoldering, symbol RESISTOR0603
Connections:
- net +5V: now also R38.2, R39.2, R40.2, R41.2, R42.2, R43.2
- net at J4.2 (Pin_2), Q6.3 (C): now also R43.1
- net at J4.3 (Pin_3), Q5.3 (C): now also R42.1
- net at J4.4 (Pin_4), Q4.3 (C): now also R41.1
- net at J4.5 (Pin_5), Q3.3 (C): now also R40.1
- net at J4.6 (Pin_6), Q2.3 (C): now also R39.1
- net at J4.7 (Pin_7), Q1.3 (C): now also R38.1
Other:
- moved on the sheet: J4, J8, R32
Changed lines of the file:
@@
 L Conn_01x08 J4
 U 1 1 5C17E262
-P 12535 7635
-F 0 "J4" H 12535 8135 50  0000 C CNN
-F 1 "Conn_01x10" H 12535 7035 50  0001 C CNN
-F 2 "Connectors_JST:JST_EH_B08B-EH-A_08x2.50mm_Straight" H 12535 7635 50  0001 C CNN
-F 3 "" H 12535 7635 50  0001 C CNN
-	1    12535 7635
+P 12835 7635
+F 0 "J4" H 12835 8135 50  0000 C CNN
+F 1 "Conn_01x10" H 12835 7035 50  0001 C CNN
+F 2 "Connectors_JST:JST_EH_B08B-EH-A_08x2.50mm_Straight" H 12835 7635 50  0001 C CNN
+F 3 "" H 12835 7635 50  0001 C CNN
+	1    12835 7635
 	1    0    0    -1
 $EndComp
@@
 L GND #PWR08
 U 1 1 5C183C5A
-P 12335 8035
-F 0 "#PWR08" H 12335 7785 50  0001 C CNN
-F 1 "GND" H 12360 7855 50  0000 C CNN
-F 2 "" H 12335 8035 50  0001 C CNN
-F 3 "" H 12335 8035 50  0001 C CNN
-	1    12335 8035
+P 12635 8035
+F 0 "#PWR08" H 12635 7785 50  0001 C CNN
+F 1 "GND" H 12660 7855 50  0000 C CNN
+F 2 "" H 12635 8035 50  0001 C CNN
+F 3 "" H 12635 8035 50  0001 C CNN
+	1    12635 8035
 	1    0    0    -1
 $EndComp
@@
 L +5V #PWR09
 U 1 1 5C1840DB
-P 12335 7335
-F 0 "#PWR09" H 12335 7185 50  0001 C CNN
-F 1 "+5V" H 12370 7535 50  0000 C CNN
-F 2 "" H 12335 7335 50  0001 C CNN
-F 3 "" H 12335 7335 50  0001 C CNN
-	1    12335 7335
+P 12635 7335
+F 0 "#PWR09" H 12635 7185 50  0001 C CNN
+F 1 "+5V" H 12670 7535 50  0000 C CNN
+F 2 "" H 12635 7335 50  0001 C CNN
+F 3 "" H 12635 7335 50  0001 C CNN
+	1    12635 7335
 	1    0    0    -1
 $EndComp
@@
 L Conn_01x06 J8
 U 1 1 5C1CF9E3
-P 8145 7740
-F 0 "J8" H 8145 8240 50  0000 C CNN
-F 1 "Conn_01x10" H 8145 7140 50  0001 C CNN
-F 2 "Connectors_JST:JST_EH_B06B-EH-A_06x2.50mm_Straight" H 8145 7740 50  0001 C CNN
-F 3 "" H 8145 7740 50  0001 C CNN
-	1    8145 7740
+P 8335 7740
+F 0 "J8" H 8335 8240 50  0000 C CNN
+F 1 "Conn_01x10" H 8335 7140 50  0001 C CNN
+F 2 "Connectors_JST:JST_EH_B06B-EH-A_06x2.50mm_Straight" H 8335 7740 50  0001 C CNN
+F 3 "" H 8335 7740 50  0001 C CNN
+	1    8335 7740
 	1    0    0    -1
 $EndComp
@@
 L +5V #PWR026
 U 1 1 5C1CFA13
-P 7945 7540
-F 0 "#PWR026" H 7945 7390 50  0001 C CNN
-F 1 "+5V" H 7980 7740 50  0000 C CNN
-F 2 "" H 7945 7540 50  0001 C CNN
-F 3 "" H 7945 7540 50  0001 C CNN
-	1    7945 7540
+P 8135 7540
+F 0 "#PWR026" H 8135 7390 50  0001 C CNN
+F 1 "+5V" H 8170 7740 50  0000 C CNN
+F 2 "" H 8135 7540 50  0001 C CNN
+F 3 "" H 8135 7540 50  0001 C CNN
+	1    8135 7540
 	1    0    0    -1
 $EndComp
@@
 L RESISTOR0603 R32
 U 1 1 5C1AFE11
-P 12135 8035
-F 0 "R32" H 12190 8190 45  0000 L BNN
-F 1 "0" H 12075 8190 45  0000 L BNN
-F 2 "Capacitors_SMD:C_0603_HandSoldering" H 12135 8185 20  0001 C CNN
-F 3 "" H 12135 8035 60  0001 C CNN
-F 4 " " V 12210 8210 60  0000 C CNN "Поле4"
-	1    12135 8035
+P 12340 8035
+F 0 "R32" H 12395 8190 45  0000 L BNN
+F 1 "0" H 12280 8190 45  0000 L BNN
+F 2 "Capacitors_SMD:C_0603_HandSoldering" H 12340 8185 20  0001 C CNN
+F 3 "" H 12340 8035 60  0001 C CNN
+F 4 " " V 12415 8210 60  0000 C CNN "Поле4"
+	1    12340 8035
 	-1   0    0    1
 $EndComp
@@
 	4270 3985 4135 3985
 Wire Wire Line
-	4270 4440 4270 2585
+	4270 2585 4270 4440
 Wire Wire Line
 	4270 3285 4135 3285
@@
 Connection ~ 4705 7995
 Wire Wire Line
-	11935 7535 12335 7535
-Wire Wire Line
-	12335 7635 11535 7635
-Wire Wire Line
-	12335 7735 11135 7735
-Wire Wire Line
-	10735 7835 12335 7835
-Wire Wire Line
-	12335 7935 10335 7935
+	11935 7535 12635 7535
+Wire Wire Line
+	11535 7635 12635 7635
+Wire Wire Line
+	11135 7735 12635 7735
+Wire Wire Line
+	10735 7835 12635 7835
+Wire Wire Line
+	10335 7935 12635 7935
 Wire Wire Line
 	9935 7935 9935 8300
 Wire Wire Line
-	11935 8300 9935 8300
-Wire Wire Line
-	11935 7435 11935 8300
+	9935 8300 11935 8300
+Wire Wire Line
+	11935 8300 11935 7435
 Wire Wire Line
 	10335 7835 10335 8300
@@
 	8860 5020 9050 5020
 Wire Wire Line
-	7945 7640 7945 7640
-Wire Wire Line
-	7945 7740 7545 7740
-Wire Wire Line
-	7145 7840 7945 7840
-Wire Wire Line
-	7945 7940 6745 7940
+	8135 7640 7945 7640
+Wire Wire Line
+	8135 7740 7545 7740
+Wire Wire Line
+	7145 7840 8135 7840
+Wire Wire Line
+	8135 7940 6745 7940
 Wire Wire Line
 	6345 7940 6345 8305
 Wire Wire Line
-	6345 8305 7945 8305
+	6345 8305 8135 8305
 Wire Wire Line
 	6745 7840 6745 8305
@@
 	7745 7140 7745 7340
 Wire Wire Line
-	7945 8305 7945 8040
-Wire Wire Line
 	8630 5420 8760 5420
 Wire Wire Line
@@
 Connection ~ 5290 6965
 $Comp
-L +3.3VA #PWR?
+L +3.3VA #PWR030
 U 1 1 5C391CA3
 P 5290 6940
-F 0 "#PWR?" H 5290 6790 50  0001 C CNN
+F 0 "#PWR030" H 5290 6790 50  0001 C CNN
 F 1 "+3.3VA" H 5290 7080 50  0000 C CNN
 F 2 "" H 5290 6940 50  0001 C CNN
@@
 $EndComp
 NoConn ~ 8630 2520
+$Comp
+L RESISTOR0603 R43
+U 1 1 5CA11209
+P 12565 8630
+F 0 "R43" V 12440 8705 45  0000 L BNN
+F 1 "1k" V 12540 8705 45  0000 L BNN
+F 2 "Capacitors_SMD:C_0603_HandSoldering" H 12565 8780 20  0001 C CNN
+F 3 "" H 12565 8630 60  0001 C CNN
+F 4 " " V 12640 8805 60  0000 C CNN "Поле4"
+	1    12565 8630
+	0    1    1    0
+$EndComp
+Wire Wire Line
+	12335 7435 12635 7435
+Wire Wire Line
+	12140 8035 11935 8035
+Wire Wire Line
+	12635 8035 12540 8035
+$Comp
+L RESISTOR0603 R42
+U 1 1 5CA133C1
+P 12070 8630
+F 0 "R42" V 11945 8705 45  0000 L BNN
+F 1 "1k" V 12045 8705 45  0000 L BNN
+F 2 "Capacitors_SMD:C_0603_HandSoldering" H 12070 8780 20  0001 C CNN
+F 3 "" H 12070 8630 60  0001 C CNN
+F 4 " " V 12145 8805 60  0000 C CNN "Поле4"
+	1    12070 8630
+	0    1    1    0
+$EndComp
+$Comp
+L RESISTOR0603 R41
+U 1 1 5CA170EF
+P 11720 8630
+F 0 "R41" V 11595 8705 45  0000 L BNN
+F 1 "1k" V 11695 8705 45  0000 L BNN
+F 2 "Capacitors_SMD:C_0603_HandSoldering" H 11720 8780 20  0001 C CNN
+F 3 "" H 11720 8630 60  0001 C CNN
+F 4 " " V 11795 8805 60  0000 C CNN "Поле4"
+	1    11720 8630
+	0    1    1    0
+$EndComp
+$Comp
+L RESISTOR0603 R40
+U 1 1 5CA17279
+P 11340 8630
+F 0 "R40" V 11215 8705 45  0000 L BNN
+F 1 "1k" V 11315 8705 45  0000 L BNN
+F 2 "Capacitors_SMD:C_0603_HandSoldering" H 11340 8780 20  0001 C CNN
+F 3 "" H 11340 8630 60  0001 C CNN
+F 4 " " V 11415 8805 60  0000 C CNN "Поле4"
+	1    11340 8630
+	0    1    1    0
+$EndComp
+$Comp
+L RESISTOR0603 R39
+U 1 1 5CA1740C
+P 10945 8630
+F 0 "R39" V 10820 8705 45  0000 L BNN
+F 1 "1k" V 10920 8705 45  0000 L BNN
+F 2 "Capacitors_SMD:C_0603_HandSoldering" H 10945 8780 20  0001 C CNN
+F 3 "" H 10945 8630 60  0001 C CNN
+F 4 " " V 11020 8805 60  0000 C CNN "Поле4"
+	1    10945 8630
+	0    1    1    0
+$EndComp
+$Comp
+L RESISTOR0603 R38
+U 1 1 5CA1780C
+P 10445 8625
+F 0 "R38" V 10320 8700 45  0000 L BNN
+F 1 "1k" V 10420 8700 45  0000 L BNN
+F 2 "Capacitors_SMD:C_0603_HandSoldering" H 10445 8775 20  0001 C CNN
+F 3 "" H 10445 8625 60  0001 C CNN
+F 4 " " V 10520 8800 60  0000 C CNN "Поле4"
+	1    10445 8625
+	0    1    1    0
+$EndComp
+Wire Wire Line
+	10445 8425 10445 7935
+Connection ~ 10445 7935
+Wire Wire Line
+	10945 8430 10945 7835
+Connection ~ 10945 7835
+Wire Wire Line
+	11720 8430 11720 7635
+Connection ~ 11720 7635
+Wire Wire Line
+	12070 8430 12070 7535
+Connection ~ 12070 7535
+Wire Wire Line
+	12565 8430 12565 7435
+Connection ~ 12565 7435
+Wire Wire Line
+	10445 8825 10445 8965
+Wire Wire Line
+	10445 8965 12565 8965
+Wire Wire Line
+	12565 8965 12565 8830
+Wire Wire Line
+	10945 8830 10945 8965
+Wire Wire Line
+	10945 8965 10940 8965
+Connection ~ 10940 8965
+Wire Wire Line
+	11340 8830 11340 8965
+Connection ~ 11340 8965
+Wire Wire Line
+	11720 8830 11720 8965
+Connection ~ 11720 8965
+Wire Wire Line
+	12070 8830 12070 8965
+Connection ~ 12070 8965
+$Comp
+L +5V #PWR031
+U 1 1 5CA19E67
+P 12315 8890
+F 0 "#PWR031" H 12315 8740 50  0001 C CNN
+F 1 "+5V" H 12350 9090 50  0000 C CNN
+F 2 "" H 12315 8890 50  0001 C CNN
+F 3 "" H 12315 8890 50  0001 C CNN
+	1    12315 8890
+	1    0    0    -1
+$EndComp
+Wire Wire Line
+	12315 8890 12315 8965
+Wire Wire Line
+	12315 8965 12310 8965
+Connection ~ 12310 8965
+Wire Wire Line
+	8135 8305 8135 8040
+Wire Wire Line
+	11340 8430 11340 7735
+Connection ~ 11340 7735
 $EndSCHEMATC

Commit message: update
Parts:
- added R44: 0, Capacitors_SMD:C_0603_HandSoldering, symbol RESISTOR0603
- Y1: Поле4 125MHz -> 40MHz
Connections:
- net +5V: now also R44.1; no longer R38.2, R39.2, R40.2, R41.2, R42.2, R43.2
- new net: R38.2, R39.2, R40.2, R41.2, R42.2, R43.2, R44.2
