File: schematic3/rpi_cpld.sch (KiCad schematic (older format))
At the start: 88 parts, among them J1 CONN_02, J2 RPi_Hat-rescue_RPi_GPIO, J3 , J4 Conn_01x10, J5 UART, J6 , J7 I2C, J8 Conn_01x10, J9 , Q1 BC817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

Commit message: update
Parts:
- removed J6: (no value), Connector_PinHeader_2.54mm:PinHeader_2x05_P2.54mm_Vertical, symbol rpi_cpld-rescue:Conn_01x10
- added J? (x2): Conn_02x07_Odd_Even, symbol Connector_Generic:Conn_02x07_Odd_Even
Connections:
- wire segments 226 -> 220
Changed lines of the file:
@@
 GNDR
-$Comp
-L rpi_cpld-rescue:Conn_01x10 J6
-U 1 1 5C1B990C
-P 9250 5020
-F 0 "J6" H 9050 5820 45  0000 L BNN
-F 1 " " H 9050 4870 45  0000 L BNN
-F 2 "Connector_PinHeader_2.54mm:PinHeader_2x05_P2.54mm_Vertical" H 9250 5920 20  0000 C CNN
-F 3 "" H 9250 5020 50  0001 C CNN
-	1    9250 5020
-	1    0    0    -1
-$EndComp
 $Comp
 L rpi_cpld-rescue:GNDA #PWR018
 U 1 1 5C1BA852
-P 9050 4620
-F 0 "#PWR018" H 9050 4370 50  0001 C CNN
-F 1 "GNDA" H 9050 4470 50  0000 C CNN
-F 2 "" H 9050 4620 50  0001 C CNN
-F 3 "" H 9050 4620 50  0001 C CNN
-	1    9050 4620
+P 10250 4900
+F 0 "#PWR018" H 10250 4650 50  0001 C CNN
+F 1 "GNDA" H 10250 4750 50  0000 C CNN
+F 2 "" H 10250 4900 50  0001 C CNN
+F 3 "" H 10250 4900 50  0001 C CNN
+	1    10250 4900
 	1    0    0    1
 $EndComp
@@
 L rpi_cpld-rescue:+3.3VA #PWR019
 U 1 1 5C1BABE1
-P 9050 4720
-F 0 "#PWR019" H 9050 4570 50  0001 C CNN
-F 1 "+3.3VA" V 9050 4970 50  0000 C CNN
-F 2 "" H 9050 4720 50  0001 C CNN
-F 3 "" H 9050 4720 50  0001 C CNN
-	1    9050 4720
+P 9750 4900
+F 0 "#PWR019" H 9750 4750 50  0001 C CNN
+F 1 "+3.3VA" V 9750 5150 50  0000 C CNN
+F 2 "" H 9750 4900 50  0001 C CNN
+F 3 "" H 9750 4900 50  0001 C CNN
+	1    9750 4900
 	0    -1   1    0
 $EndComp
@@
 Connection ~ 6680 1075
 Wire Wire Line
-	9050 4820 8860 4820
-Wire Wire Line
-	8860 4820 8760 4920
-Wire Wire Line
-	8760 4920 8630 4920
-Wire Wire Line
-	8630 4820 8755 4820
-Wire Wire Line
-	8755 4820 8855 4920
-Wire Wire Line
-	8855 4920 9050 4920
-Wire Wire Line
 	4490 6965 4855 6965
 Wire Wire Line
@@
 Wire Wire Line
 	10445 8965 11340 8965
+$Comp
+L Connector_Generic:Conn_02x07_Odd_Even J?
+U 1 1 5CA7030B
+P 9950 5200
+F 0 "J?" H 10000 5650 50  0000 C CNN
+F 1 "Conn_02x07_Odd_Even" H 10015 5670 50  0001 C CNN
+F 2 "" H 9950 5200 50  0001 C CNN
+F 3 "~" H 9950 5200 50  0001 C CNN
+	1    9950 5200
+	1    0    0    -1
+$EndComp
+$Comp
+L Connector_Generic:Conn_02x07_Odd_Even J?
+U 1 1 5CA71A3D
+P 10565 2955
+F 0 "J?" H 10630 3500 50  0000 C CNN
+F 1 "Conn_02x07_Odd_Even" H 10630 3400 50  0000 C CNN
+F 2 "" H 10565 2955 50  0001 C CNN
+F 3 "~" H 10565 2955 50  0001 C CNN
+	1    10565 2955
+	1    0    0    -1
+$EndComp
 $EndSCHEMATC
